File: kicad/Eurorack-PT2399-Delay.kicad_sch (KiCad schematic)
At the start: 97 parts, among them J1 EuroPower_JST_3P, J2 EURO_PWR_16P, J3 Main_in, J4 Aux_in, J5 Time_CV_in, J6 Wet_out_1, J7 Wet_out_2, J8 dry_out, Q1 BC547, Q2 BC547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

Commit message: Schematic rev 0.1.0 update
Connections:
- net GND: now also U4.3 (+); no longer U4.2 (-)
- net at C22.1, R10.2, R8.2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: now also U4.2 (-); no longer U4.3 (+)
Changed lines of the file:
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@@
     )
   )
-  (symbol (lib_id "Amplifier_Operational:TL074") (at 108.585 46.355 0) (unit 1)
+  (symbol (lib_id "Amplifier_Operational:TL074") (at 108.585 46.355 0) (mirror x) (unit 1)
     (in_bom yes) (on_board yes) (dnp no)
-    (property "Reference" "U4" (at 110.49 50.165 0)
+    (property "Reference" "U4" (at 110.49 53.34 0)
       (effects (font (size 1.27 1.27)))
     )
-    (property "Value" "TL074" (at 110.49 52.705 0)
+    (property "Value" "TL074" (at 110.49 50.8 0)
       (effects (font (size 1.27 1.27)))
     )
-    (property "Footprint" "" (at 107.315 43.815 0)
+    (property "Footprint" "" (at 107.315 48.895 0)
       (effects (font (size 1.27 1.27)) hide)
     )
-    (property "Datasheet" "http://www.ti.com/lit/ds/symlink/tl071.pdf" (at 109.855 41.275 0)
+    (property "Datasheet" "http://www.ti.com/lit/ds/symlink/tl071.pdf" (at 109.855 51.435 0)
       (effects (font (size 1.27 1.27)) hide)
     )

Commit message: Add schematic rev 0.1.1
Parts:
- added RV8: 100K, symbol Device:R_Potentiometer
- R9: value 100K -> 39K
- RV6: value 100K -> 200K
Connections:
- net GND: now also RV8.1
- net at C18.1, R11.1: now also RV8.2; no longer J3.T
- new net: J3.T, RV8.3
Other:
- note added: "Rev 0.1.1 Add RV8 audio input attenuation knob. Change output gain trimmer RV6 to 200K. Change feedback resistor R24 to 220K."
- moved on the sheet: J3
Changed lines of the file:
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@@
     (title "Eurorack PT2399 Delay")
     (date "2024-02-23")
-    (rev "0.1.0")
+    (rev "0.1.1")
     (company "DIYSynthMNL")
   )
@@
   (junction (at 203.2 259.08) (diameter 0) (color 0 0 0 0)
   )
+  (junction (at 75.565 39.37) (diameter 0) (color 0 0 0 0)
+  )
   (junction (at 185.42 114.935) (diameter 0) (color 0 0 0 0)
   )
@@
   (junction (at 100.965 39.37) (diameter 0) (color 0 0 0 0)
   )
-  (junction (at 75.565 39.37) (diameter 0) (color 0 0 0 0)
-  )
   (junction (at 162.56 178.435) (diameter 0) (color 0 0 0 0)
   )
@@
   (no_connect (at 56.515 254))
   (no_connect (at 67.945 92.075))
-  (no_connect (at 69.215 36.83))
+  (no_connect (at 52.705 36.83))
   (no_connect (at 79.375 254))
   (no_connect (at 332.74 107.95))
@@
     (stroke (width 0) (type default))
   )
+  (wire (pts (xy 52.705 41.91) (xy 52.705 42.545))
+    (stroke (width 0) (type default))
+  )
   (wire (pts (xy 227.33 111.125) (xy 227.33 108.585))
     (stroke (width 0) (type default))
@@
     (stroke (width 0) (type default))
   )
-  (wire (pts (xy 120.65 112.395) (xy 127.635 112.395))
+  (wire (pts (xy 58.42 39.37) (xy 52.705 39.37))
     (stroke (width 0) (type default))
   )
-  (wire (pts (xy 166.37 191.77) (xy 166.37 189.23))
+  (wire (pts (xy 68.58 39.37) (xy 75.565 39.37))
+    (stroke (width 0) (type default))
+  )
+  (wire (pts (xy 120.65 112.395) (xy 127.635 112.395))
     (stroke (width 0) (type default))
   )
-  (wire (pts (xy 69.215 39.37) (xy 75.565 39.37))
+  (wire (pts (xy 166.37 191.77) (xy 166.37 189.23))
     (stroke (width 0) (type default))
   )
@@
     (stroke (width 0) (type default))
   )
+  (wire (pts (xy 58.42 41.91) (xy 58.42 39.37))
+    (stroke (width 0) (type default))
+  )
   (wire (pts (xy 227.33 121.285) (xy 211.455 121.285))
     (stroke (width 0) (type default))
@@
     (stroke (width 0) (type default))
   )
+  (wire (pts (xy 68.58 45.72) (xy 68.58 39.37))
+    (stroke (width 0) (type default))
+  )
   (wire (pts (xy 329.565 170.18) (xy 326.39 170.18))
     (stroke (width 0) (type default))
@@
     (stroke (width 0) (type default))
   )
+  (wire (pts (xy 68.58 45.72) (xy 62.23 45.72))
+    (stroke (width 0) (type default))
+  )
   (wire (pts (xy 127.635 247.65) (xy 127.635 245.11))
     (stroke (width 0) (type default))
@@
     (effects (font (size 1.27 1.27)) (justify left bottom))
   )
+  (text "Rev 0.1.1\nAdd RV8 audio input attenuation knob.\nChange output gain trimmer RV6 to 200K.\nChange feedback resistor R24 to 220K.\n"
+    (at 321.945 265.43 0)
+    (effects (font (size 1.27 1.27)) (justify left bottom))
+  )
   (text "Op Amp Power" (at 240.03 229.87 0)
     (effects (font (size 1.27 1.27)) (justify left bottom))
@@
     )
   )
+  (symbol (lib_id "Device:R_Potentiometer") (at 58.42 45.72 0) (mirror x) (unit 1)
+    (in_bom yes) (on_board yes) (dnp no)
+    (property "Reference" "RV8" (at 64.77 47.625 0)
+      (effects (font (size 1.27 1.27)) (justify right))
+    )
+    (property "Value" "100K" (at 66.04 50.165 0)
+      (effects (font (size 1.27 1.27)) (justify right))
+    )
+    (property "Footprint" "" (at 58.42 45.72 0)
+      (effects (font (size 1.27 1.27)) hide)
+    )
+    (property "Datasheet" "~" (at 58.42 45.72 0)
+      (effects (font (size 1.27 1.27)) hide)
+    )
+    (pin "3")
+    (pin "2")
+    (pin "1")
+    (instances
+      (project "Eurorack-PT2399-Delay"
+        (path "/14ea4fda-251e-4d7d-a5a0-88726fa92ee2"
+          (reference "RV8") (unit 1)
+        )
+      )
+    )
+  )
   (symbol (lib_id "Device:R") (at 131.445 100.965 90) (unit 1)
     (in_bom yes) (on_board yes) (dnp no)
@@
     )
   )
+  (symbol (lib_id "power:GND") (at 58.42 49.53 0) (unit 1)
+    (in_bom yes) (on_board yes) (dnp no) (fields_autoplaced)
+    (property "Reference" "#PWR056" (at 58.42 55.88 0)
+      (effects (font (size 1.27 1.27)) hide)
+    )
+    (property "Value" "GND" (at 58.42 54.61 0)
+      (effects (font (size 1.27 1.27)))
+    )
+    (property "Footprint" "" (at 58.42 49.53 0)
+      (effects (font (size 1.27 1.27)) hide)
+    )
+    (property "Datasheet" "" (at 58.42 49.53 0)
+      (effects (font (size 1.27 1.27)) hide)
+    )
+    (pin "1")
+    (instances
+      (project "Eurorack-PT2399-Delay"
+        (path "/14ea4fda-251e-4d7d-a5a0-88726fa92ee2"
+          (reference "#PWR056") (unit 1)
+        )
+      )
+      (project "Electric Druid VCDO1"
+        (path "/1a79e409-2950-446e-9b6e-16f6bf0a888d"
+          (reference "#PWR?") (unit 1)
+        )
+        (path "/1a79e409-2950-446e-9b6e-16f6bf0a888d/940513db-8445-4e70-8397-130f22045b59"
+          (reference "#PWR?") (unit 1)
+        )
+      )
+      (project "3340-VCO"
+        (path "/aedb3b78-1db1-4bb8-b4e7-c509f764608a"
+          (reference "#PWR045") (unit 1)
+        )
+        (path "/aedb3b78-1db1-4bb8-b4e7-c509f764608a/7052fdfb-ea3f-4ad0-aa23-37dd6b189892"
+          (reference "#PWR045") (unit 1)
+        )
+      )
+    )
+  )
   (symbol (lib_id "Transistor_BJT:BC547") (at 213.995 93.98 0) (mirror y) (unit 1)
     (in_bom yes) (on_board yes) (dnp no)
@@
       (effects (font (size 1.27 1.27)))
     )
-    (property "Value" "100K" (at 109.22 39.37 90)
+    (property "Value" "39K" (at 109.22 39.37 90)
       (effects (font (size 1.27 1.27)))
     )
@@
     )
   )
-  (symbol (lib_id "power:GND") (at 69.215 41.91 0) (unit 1)
+  (symbol (lib_id "power:GND") (at 52.705 42.545 0) (unit 1)
     (in_bom yes) (on_board yes) (dnp no) (fields_autoplaced)
-    (property "Reference" "#PWR021" (at 69.215 48.26 0)
+    (property "Reference" "#PWR021" (at 52.705 48.895 0)
       (effects (font (size 1.27 1.27)) hide)
     )
-    (property "Value" "GND" (at 69.215 46.99 0)
+    (property "Value" "GND" (at 52.705 47.625 0)
       (effects (font (size 1.27 1.27)))
     )
-    (property "Footprint" "" (at 69.215 41.91 0)
+    (property "Footprint" "" (at 52.705 42.545 0)
       (effects (font (size 1.27 1.27)) hide)
     )
-    (property "Datasheet" "" (at 69.215 41.91 0)
+    (property "Datasheet" "" (at 52.705 42.545 0)
       (effects (font (size 1.27 1.27)) hide)
     )
@@
     )
   )
-  (symbol (lib_id "DIYSynthMNL:PJ3001F") (at 64.135 39.37 0) (mirror x) (unit 1)
+  (symbol (lib_id "DIYSynthMNL:PJ3001F") (at 47.625 39.37 0) (mirror x) (unit 1)
     (in_bom yes) (on_board yes) (dnp no) (fields_autoplaced)
-    (property "Reference" "J3" (at 58.42 37.465 0)
+    (property "Reference" "J3" (at 41.91 37.465 0)
       (effects (font (size 1.27 1.27)) (justify right))
     )
-    (property "Value" "Main_in" (at 58.42 40.005 0)
+    (property "Value" "Main_in" (at 41.91 40.005 0)
       (effects (font (size 1.27 1.27)) (justify right))
     )
-    (property "Footprint" "DIYSynthMNL:AudioJack_3.5mm_long_pads" (at 64.135 31.75 0)
+    (property "Footprint" "DIYSynthMNL:AudioJack_3.5mm_long_pads" (at 47.625 31.75 0)
       (effects (font (size 1.27 1.27)) hide)
     )
-    (property "Datasheet" "~" (at 64.135 39.37 0)
+    (property "Datasheet" "~" (at 47.625 39.37 0)
       (effects (font (size 1.27 1.27)) hide)
     )
@@
       (effects (font (size 1.27 1.27)))
     )
-    (property "Value" "100K" (at 250.19 182.245 0)
+    (property "Value" "200K" (at 250.19 182.245 0)
       (effects (font (size 1.27 1.27)))
     )
